File: atmega-demos/avr_usbasp/circuit/kicad/usbasploader/usbasploader.kicad_pcb (KiCad board)
At the start: 2 copper layers, 28.9 x 35.4 mm, 21 parts, among them J1 Conn_01x06_Pin, J2 USB_B_Mini, SW1 SW_Push, SW2 SW_Push, U1 ATmega8A-A, Y1 12MHz

Commit message: USBASP Loader PCB
Parts:
- added C1: 100n, Capacitor_SMD:C_0805_2012Metric_Pad1.18x1.45mm_HandSolder, F.Cu at (105.4, 68.0)
- D4, D5: value 3V3 -> 3V6
- renumbered C1 to C2, C2 to C3
Routing:
- net VCC: track 131.0 -> 132.5 mm, vias 2 -> 3
- net GND: track 58.7 -> 60.1 mm, vias 7 -> 8
- removed copper zone on F.Cu, net (none)
